File: OdysseyDaughterCardVertSyncGenerator.kicad_pcb (KiCad board)
At the start: 2 copper layers, 29 x 46.6 mm, 13 parts, among them Q1 2N3904, Q2 2N3906, Q3 2N3904, X1 OdysseyDaughterCard

Commit message: Bump rev number and regenerate gerbers
Other:
- board text added: "Daughter Card Vertical Sync Generator 8-18-2018 r0.2 University of Pittsburgh Odyssey Restoration Project"
- board text removed: "Daughter Card Vertical Sync Generator 6-7-2018 r0.1 University of Pittsburgh Odyssey Restoration Project"
Changed lines of the file:
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@@
   (title_block
     (title "Odyssey Daughter Card Vertical Sync Generator")
-    (date 2018-06-07)
-    (rev 0.1)
+    (date 2018-08-18)
+    (rev 0.2)
     (company "University of Pittsburgh - Odyssey Restoration Project")
     (comment 1 "Levi Burner")
@@
   (gr_line (start 126.175 124.3) (end 126.175 123.1) (layer Edge.Cuts) (width 0.15))
   (gr_line (start 122.425 124.3) (end 126.175 124.3) (layer Edge.Cuts) (width 0.15))
-  (gr_text "Daughter Card Vertical Sync Generator\n6-7-2018 r0.1\nUniversity of Pittsburgh\nOdyssey Restoration Project" (at 129.032 80.264 -90) (layer F.SilkS)
+  (gr_text "Daughter Card Vertical Sync Generator\n8-18-2018 r0.2\nUniversity of Pittsburgh\nOdyssey Restoration Project" (at 129.032 80.264 -90) (layer F.SilkS)
     (effects (font (size 1.2 1.2) (thickness 0.2)) (justify left))
   )
