File: OdysseyDaughterCardVertSyncGenerator.sch (KiCad schematic (older format))
At the start: 13 parts, among them Q1 2N3904, Q2 2N3906, Q3 2N3904, X1 OdysseyDaughterCard

Commit message: Add note about BLAK vs BK12 console revisions
Parts:
- X1: symbol Odyssey_Daughter_Card:OdysseyDaughterCard -> OdysseyDaughterCardVertSyncGenerator-rescue:OdysseyDaughterCard-Odyssey_Daughter_Card
Other:
- note added: "This is BLAK version, not comptabile with BK12 Odysseys\nSee "How to Repair Video Games" by Robert Goodman pg. 138-141\nfor BK12 schematic"
Changed lines of the file:
@@
 EESchema Schematic File Version 4
 LIBS:OdysseyDaughterCardVertSyncGenerator-cache
-EELAYER 26 0
+EELAYER 29 0
 EELAYER END
 $Descr A4 11693 8268
@@
 $EndDescr
 $Comp
-L Odyssey_Daughter_Card:OdysseyDaughterCard X1
+L OdysseyDaughterCardVertSyncGenerator-rescue:OdysseyDaughterCard-Odyssey_Daughter_Card X1
 U 1 1 5B0D981F
 P 5700 3700
@@
 NoConn ~ 5950 3800
 NoConn ~ 5950 3900
+Text Notes 7550 4550 0    60   ~ 0
+This is BLAK version, not comptabile with BK12 Odysseys\nSee "How to Repair Video Games" by Robert Goodman pg. 138-141\nfor BK12 schematic
 $EndSCHEMATC
