File: OdysseyDaughterCardFlipFlop/OdysseyDaughterCardFlipFlop.kicad_sch (KiCad schematic)
At the start: 17 parts, among them J1 Conn_01x02, Q1 2N3906, Q2 2N3906, Q3 BC547C, Q4 BC547C, X1 OdysseyDaughterCard

Commit message: OdysseyDaughterCardFlipFlop wider transistor footprint, logo, pours, pdfs, images, 3d model
Parts:
- Q1, Q2, Q3, Q4: footprint Package_TO_SOT_THT:TO-92_Inline -> Package_TO_SOT_THT:TO-92_Inline_Wide
Other:
- company: University of Pittsburgh - Odyssey Restoration Project -> University of Pittsburgh - OdysseyNow
