File: OdysseyDaughterCardTemplate/OdysseyDaughterCardTemplate.kicad_pcb (KiCad board)
At the start: 2 copper layers, 47.8 x 46.6 mm, 1 part, among them X1 OdysseyDaughterCard

Commit message: OdysseyDaughterCardTemplate: Open and close in KiCad 6, fix symbol library pathwq
Other:
- net class Default removed
Changed lines of the file:
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@@
-(kicad_pcb (version 20171130) (host pcbnew "(2017-12-21 revision 23d71cfa9)-makepkg")
+(kicad_pcb (version 20211014) (generator pcbnew)
   (general
     (thickness 1.6)
-    (drawings 13)
-    (tracks 0)
-    (zones 0)
-    (modules 1)
-    (nets 11)
   )
-  (page A4)
+  (paper "A4")
   (title_block
     (title "Odyssey Daughter Card Template")
-    (date 2018-05-29)
-    (rev 0.1)
+    (date "2018-05-29")
+    (rev "0.1")
     (company "University of Pittsburgh - Odyssey Restoration Project")
     (comment 1 "Levi Burner")
   )
   (layers
-    (0 F.Cu signal)
-    (31 B.Cu signal)
-    (32 B.Adhes user)
-    (33 F.Adhes user)
-    (34 B.Paste user)
-    (35 F.Paste user)
-    (36 B.SilkS user)
-    (37 F.SilkS user)
-    (38 B.Mask user)
-    (39 F.Mask user)
-    (40 Dwgs.User user)
-    (41 Cmts.User user)
-    (42 Eco1.User user)
-    (43 Eco2.User user)
-    (44 Edge.Cuts user)
-    (45 Margin user)
-    (46 B.CrtYd user)
-    (47 F.CrtYd user)
-    (48 B.Fab user)
-    (49 F.Fab user)
+    (0 "F.Cu" signal)
+    (31 "B.Cu" signal)
+    (32 "B.Adhes" user "B.Adhesive")
+    (33 "F.Adhes" user "F.Adhesive")
+    (34 "B.Paste" user)
+    (35 "F.Paste" user)
+    (36 "B.SilkS" user "B.Silkscreen")
+    (37 "F.SilkS" user "F.Silkscreen")
+    (38 "B.Mask" user)
+    (39 "F.Mask" user)
+    (40 "Dwgs.User" user "User.Drawings")
+    (41 "Cmts.User" user "User.Comments")
+    (42 "Eco1.User" user "User.Eco1")
+    (43 "Eco2.User" user "User.Eco2")
+    (44 "Edge.Cuts" user)
+    (45 "Margin" user)
+    (46 "B.CrtYd" user "B.Courtyard")
+    (47 "F.CrtYd" user "F.Courtyard")
+    (48 "B.Fab" user)
+    (49 "F.Fab" user)
   )
   (setup
-    (last_trace_width 0.25)
-    (user_trace_width 2.5)
-    (trace_clearance 0.2)
-    (zone_clearance 0.508)
-    (zone_45_only no)
-    (trace_min 0.2)
-    (segment_width 0.2)
-    (edge_width 0.15)
-    (via_size 0.8)
-    (via_drill 0.4)
-    (via_min_size 0.4)
-    (via_min_drill 0.3)
-    (uvia_size 0.3)
-    (uvia_drill 0.1)
-    (uvias_allowed no)
-    (uvia_min_size 0.2)
-    (uvia_min_drill 0.1)
-    (pcb_text_width 0.3)
-    (pcb_text_size 1.5 1.5)
-    (mod_edge_width 0.15)
-    (mod_text_size 1 1)
-    (mod_text_width 0.15)
-    (pad_size 1.524 1.524)
-    (pad_drill 0.762)
     (pad_to_mask_clearance 0.2)
-    (aux_axis_origin 0 0)
-    (visible_elements 7FFFFFFF)
     (pcbplotparams
-      (layerselection 0x010fc_ffffffff)
+      (layerselection 0x00010fc_ffffffff)
+      (disableapertmacros false)
       (usegerberextensions false)
       (usegerberattributes false)
       (usegerberadvancedattributes false)
       (creategerberjobfile false)
+      (svguseinch false)
+      (svgprecision 6)
       (excludeedgelayer true)
-      (linewidth 0.100000)
       (plotframeref false)
       (viasonmask false)
@@
       (hpglpennumber 1)
       (hpglpenspeed 20)
-      (hpglpendiameter 15)
+      (hpglpendiameter 15.000000)
+      (dxfpolygonmode true)
+      (dxfimperialunits true)
+      (dxfusepcbnewfont true)
       (psnegative false)
       (psa4output false)
@@
       (plotvalue true)
       (plotinvisibletext false)
-      (padsonsilk false)
+      (sketchpadsonfab false)
       (subtractmaskfromsilk false)
       (outputformat 1)
@@
       (drillshape 1)
       (scaleselection 1)
-      (outputdirectory ""))
+      (outputdirectory "")
+    )
   )
   (net 0 "")
@@
   (net 9 "Net-(X1-Pad10)")
   (net 10 "Net-(X1-Pad4)")
-  (net_class Default "This is the default net class."
-    (clearance 0.2)
-    (trace_width 0.25)
-    (via_dia 0.8)
-    (via_drill 0.4)
-    (uvia_dia 0.3)
-    (uvia_drill 0.1)
-    (add_net "Net-(X1-Pad1)")
-    (add_net "Net-(X1-Pad10)")
-    (add_net "Net-(X1-Pad2)")
-    (add_net "Net-(X1-Pad3)")
-    (add_net "Net-(X1-Pad4)")
-    (add_net "Net-(X1-Pad5)")
-    (add_net "Net-(X1-Pad6)")
-    (add_net "Net-(X1-Pad7)")
-    (add_net "Net-(X1-Pad8)")
-    (add_net "Net-(X1-Pad9)")
-  )
-  (module Odyssey_Daughter_Card:Odyssey_Daughter_Card (layer F.Cu)
+  (footprint "Odyssey_Daughter_Card:Odyssey_Daughter_Card" (layer "F.Cu")
     (at 129 101)
-    (fp_text reference X1 (at 7.5 0 90) (layer B.SilkS)
+    (attr through_hole)
+    (fp_text reference "X1" (at 7.5 0 90) (layer "B.SilkS")
       (effects (font (size 1 1) (thickness 0.15)) (justify mirror))
     )
-    (fp_text value OdysseyDaughterCard (at 0 -23.25) (layer F.Fab)
+    (fp_text value "OdysseyDaughterCard" (at 0 -23.25) (layer "F.Fab")
       (effects (font (size 1 1) (thickness 0.15)))
     )
-    (fp_line (start -5 -22.25) (end 6.5 -22.25) (layer B.SilkS) (width 0.15))
-    (fp_line (start 6.5 -22.25) (end 6.5 22.25) (layer B.SilkS) (width 0.15))
-    (fp_line (start 6.5 22.25) (end -5 22.25) (layer B.SilkS) (width 0.15))
-    (pad 10 smd rect (at 0 -19.75) (size 11 3.25) (layers B.Cu B.Mask)
+    (fp_line (start 6.5 22.25) (end -5 22.25) (layer "B.SilkS") (width 0.15))
+    (fp_line (start 6.5 -22.25) (end 6.5 22.25) (layer "B.SilkS") (width 0.15))
+    (fp_line (start -5 -22.25) (end 6.5 -22.25) (layer "B.SilkS") (width 0.15))
+    (pad "1" smd rect locked (at 0 19.749992) (size 11 3.25) (layers "B.Cu" "B.Mask")
+      (net 5 "Net-(X1-Pad1)"))
+    (pad "2" smd rect locked (at 0 15.361104) (size 11 3.25) (layers "B.Cu" "B.Mask")
+      (net 6 "Net-(X1-Pad2)"))
+    (pad "3" smd rect locked (at 0 10.972216) (size 11 3.25) (layers "B.Cu" "B.Mask")
+      (net 4 "Net-(X1-Pad3)"))
+    (pad "4" smd rect locked (at 0 6.583328) (size 11 3.25) (layers "B.Cu" "B.Mask")
+      (net 10 "Net-(X1-Pad4)"))
+    (pad "5" smd rect locked (at 0 2.19444) (size 11 3.25) (layers "B.Cu" "B.Mask")
+      (net 3 "Net-(X1-Pad5)"))
+    (pad "6" smd rect locked (at 0 -2.194448) (size 11 3.25) (layers "B.Cu" "B.Mask")
+      (net 7 "Net-(X1-Pad6)"))
+    (pad "7" smd rect locked (at 0 -6.583336) (size 11 3.25) (layers "B.Cu" "B.Mask")
+      (net 2 "Net-(X1-Pad7)"))
+    (pad "8" smd rect locked (at 0 -10.972224) (size 11 3.25) (layers "B.Cu" "B.Mask")
+      (net 8 "Net-(X1-Pad8)"))
+    (pad "9" smd rect locked (at 0 -15.361112) (size 11 3.25) (layers "B.Cu" "B.Mask")
+      (net 1 "Net-(X1-Pad9)"))
+    (pad "10" smd rect locked (at 0 -19.75) (size 11 3.25) (layers "B.Cu" "B.Mask")
       (net 9 "Net-(X1-Pad10)"))
-    (pad 9 smd rect (at 0 -15.361112) (size 11 3.25) (layers B.Cu B.Mask)
-      (net 1 "Net-(X1-Pad9)"))
-    (pad 8 smd rect (at 0 -10.972224) (size 11 3.25) (layers B.Cu B.Mask)
-      (net 8 "Net-(X1-Pad8)"))
-    (pad 7 smd rect (at 0 -6.583336) (size 11 3.25) (layers B.Cu B.Mask)
-      (net 2 "Net-(X1-Pad7)"))
-    (pad 6 smd rect (at 0 -2.194448) (size 11 3.25) (layers B.Cu B.Mask)
-      (net 7 "Net-(X1-Pad6)"))
-    (pad 5 smd rect (at 0 2.19444) (size 11 3.25) (layers B.Cu B.Mask)
-      (net 3 "Net-(X1-Pad5)"))
-    (pad 4 smd rect (at 0 6.583328) (size 11 3.25) (layers B.Cu B.Mask)
-      (net 10 "Net-(X1-Pad4)"))
-    (pad 3 smd rect (at 0 10.972216) (size 11 3.25) (layers B.Cu B.Mask)
-      (net 4 "Net-(X1-Pad3)"))
-    (pad 2 smd rect (at 0 15.361104) (size 11 3.25) (layers B.Cu B.Mask)
-      (net 6 "Net-(X1-Pad2)"))
-    (pad 1 smd rect (at 0 19.749992) (size 11 3.25) (layers B.Cu B.Mask)
-      (net 5 "Net-(X1-Pad1)"))
   )
-  (gr_line (start 170.175 77.7) (end 170.175 124.3) (layer Edge.Cuts) (width 0.15))
-  (gr_line (start 126.175 77.7) (end 122.425 77.7) (layer Edge.Cuts) (width 0.15))
-  (gr_line (start 126.175 78.9) (end 126.175 77.7) (layer Edge.Cuts) (width 0.15))
-  (gr_line (start 130.775 78.9) (end 126.175 78.9) (layer Edge.Cuts) (width 0.15))
-  (gr_line (start 130.775 77.7) (end 130.775 78.9) (layer Edge.Cuts) (width 0.15))
-  (gr_line (start 170.175 77.7) (end 130.775 77.7) (layer Edge.Cuts) (width 0.15))
-  (gr_line (start 130.775 124.3) (end 170.175 124.3) (layer Edge.Cuts) (width 0.15))
-  (gr_line (start 130.775 123.1) (end 130.775 124.3) (layer Edge.Cuts) (width 0.15))
-  (gr_line (start 126.175 123.1) (end 130.775 123.1) (layer Edge.Cuts) (width 0.15))
-  (gr_line (start 126.175 124.3) (end 126.175 123.1) (layer Edge.Cuts) (width 0.15))
-  (gr_line (start 122.425 124.3) (end 126.175 124.3) (layer Edge.Cuts) (width 0.15))
-  (gr_text "Daughter Card X\n5-29-2018 r0.1\nUniversity of Pittsburgh\nOdyssey Restoration Project" (at 165.055 78.79 -90) (layer F.SilkS)
+  (gr_line (start 126.175 78.9) (end 126.175 77.7) (layer "Edge.Cuts") (width 0.15))
+  (gr_line (start 130.775 77.7) (end 130.775 78.9) (layer "Edge.Cuts") (width 0.15))
+  (gr_line (start 130.775 78.9) (end 126.175 78.9) (layer "Edge.Cuts") (width 0.15))
+  (gr_line (start 170.175 77.7) (end 170.175 124.3) (layer "Edge.Cuts") (width 0.15))
+  (gr_line (start 126.175 77.7) (end 122.425 77.7) (layer "Edge.Cuts") (width 0.15))
+  (gr_line (start 122.425 124.3) (end 122.425 77.7) (layer "Edge.Cuts") (width 0.15))
+  (gr_line (start 130.775 124.3) (end 170.175 124.3) (layer "Edge.Cuts") (width 0.15))
+  (gr_line (start 122.425 124.3) (end 126.175 124.3) (layer "Edge.Cuts") (width 0.15))
+  (gr_line (start 126.175 123.1) (end 130.775 123.1) (layer "Edge.Cuts") (width 0.15))
+  (gr_line (start 170.175 77.7) (end 130.775 77.7) (layer "Edge.Cuts") (width 0.15))
+  (gr_line (start 130.775 123.1) (end 130.775 124.3) (layer "Edge.Cuts") (width 0.15))
+  (gr_line (start 126.175 124.3) (end 126.175 123.1) (layer "Edge.Cuts") (width 0.15))
+  (gr_text "Daughter Card X\n5-29-2018 r0.1\nUniversity of Pittsburgh\nOdyssey Restoration Project" (at 165.055 78.79 -90) (layer "F.SilkS")
     (effects (font (size 1.2 1.2) (thickness 0.2)) (justify left))
   )
-  (gr_line (start 122.425 124.3) (end 122.425 77.7) (layer Edge.Cuts) (width 0.15))
 )

Commit message: OdysseyDaughterCardTemplate add logo
Parts:
- added X2: OdysseyNow_Logo, Odyssey_Daughter_Card:OdysseyNowLogo, F.Cu at (130.2, 111.6)
Other:
- board text added: "Daughter Card X 06-10-2024 r0.1 University of Pittsburgh OdysseyNow"
- board text removed: "Daughter Card X 5-29-2018 r0.1 University of Pittsburgh Odyssey Restoration Project"
