File: OdysseyDaughterCardTemplate/OdysseyDaughterCardTemplate.kicad_sch (KiCad schematic)
At the start: 1 part

Commit message: OdysseyDaughterCardTemplate add logo
Parts:
- X1: value (none) -> OdysseyDaughterCard; footprint (none) -> Odyssey_Daughter_Card:Odyssey_Daughter_Card
Other:
- company: University of Pittsburgh - Odyssey Restoration Project -> University of Pittsburgh - OdysseyNow
